Commit message: robot progress

File: lbx_robotics/src/lbx_franka_description/urdf/fr3.urdf (robot description, URDF)
Before this commit: robot fr3, 14 links, 13 joints
Links:
- link fr3_hand: geometry collision mesh filename=https://raw.githubusercontent.com/frankaemika/franka_descri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; visual mesh filename=https://raw.githubusercontent.com/frankaemika/franka_descri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
- link fr3_leftfinger: geometry collision box size=17.5e-3 15.2e-3 18.5e-3; collision box size=17.5e-3 7e-3 23.5e-3
- link fr3_link0: geometry collision mesh filename=https://raw.githubusercontent.com/frankaemika/franka_descri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; visual mesh filename=https://raw.githubusercontent.com/frankaemika/franka_descri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
- link fr3_link1: geometry collision mesh filename=https://raw.githubusercontent.com/frankaemika/franka_descri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; visual mesh filename=https://raw.githubusercontent.com/frankaemika/franka_descri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
- link fr3_link2: geometry collision mesh filename=https://raw.githubusercontent.com/frankaemika/franka_descri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; visual mesh filename=https://raw.githubusercontent.com/frankaemika/franka_descri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
- link fr3_link3: geometry collision mesh filename=https://raw.githubusercontent.com/frankaemika/franka_descri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; visual mesh filename=https://raw.githubusercontent.com/frankaemika/franka_descri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
- link fr3_link4: geometry collision mesh filename=https://raw.githubusercontent.com/frankaemika/franka_descri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; visual mesh filename=https://raw.githubusercontent.com/frankaemika/franka_descri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
- link fr3_link5: geometry collision mesh filename=https://raw.githubusercontent.com/frankaemika/franka_descri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; visual mesh filename=https://raw.githubusercontent.com/frankaemika/franka_descri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
- link fr3_link6: geometry collision mesh filename=https://raw.githubusercontent.com/frankaemika/franka_descri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; visual mesh filename=https://raw.githubusercontent.com/frankaemika/franka_descri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
- link fr3_link7: geometry collision mesh filename=https://raw.githubusercontent.com/frankaemika/franka_descri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; visual mesh filename=https://raw.githubusercontent.com/frankaemika/franka_descri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
- link fr3_rightfinger: geometry collision box size=17.5e-3 15.2e-3 18.5e-3; collision box size=17.5e-3 7e-3 23.5e-3

File: lbx_robotics/src/lbx_franka_description/urdf/fr3.urdf.xacro (robot description, xacro)
@@ -1,16 +1,37 @@
 <?xml version="1.0" encoding="utf-8"?>
 <robot xmlns:xacro="http://www.ros.org/wiki/xacro" name="fr3">
-  <!-- Import ros2_control xacro -->
-  <xacro:include filename="$(find lbx_franka_description)/urdf/fr3_ros2_control.xacro" />
   <!-- Parameters -->
   <xacro:arg name="arm_id" default="fr3" />
   <xacro:arg name="robot_ip" default="192.168.1.59" />
   <xacro:arg name="use_fake_hardware" default="false" />
-  <!-- Include the base robot URDF -->
-  <xacro:include filename="$(find lbx_franka_description)/urdf/fr3.urdf" />
-  <!-- Add ros2_control -->
-  <xacro:fr3_ros2_control
+  <xacro:arg name="hand" default="true" />
+  <xacro:arg name="gazebo" default="false" />
+  <xacro:arg name="no_prefix" default="false" />
+  <xacro:arg name="ee_id" default="franka_hand" />
+  <xacro:arg name="with_sc" default="false" />
+  <xacro:arg name="fake_sensor_commands" default="false" />
+  <xacro:arg name="gazebo_effort" default="false" />
+  <xacro:arg name="multi_arm" default="false" />
+  <!-- Include the base Franka robot description -->
+  <xacro:include filename="$(find franka_description)/robots/common/franka_robot.xacro" />
+  <!-- Create the Franka robot with ros2_control enabled -->
+  <xacro:franka_robot
     arm_id="$(arg arm_id)"
+    joint_limits="${xacro.load_yaml('$(find franka_description)/robots/fr3/joint_limits.yaml')}"
+    inertials="${xacro.load_yaml('$(find franka_description)/robots/fr3/inertials.yaml')}"
+    kinematics="${xacro.load_yaml('$(find franka_description)/robots/fr3/kinematics.yaml')}"
+    dynamics="${xacro.load_yaml('$(find franka_description)/robots/fr3/dynamics.yaml')}"
+    hand="$(arg hand)"
+    ee_id="$(arg ee_id)"
+    gazebo="$(arg gazebo)"
+    with_sc="$(arg with_sc)"
+    ros2_control="true"
     robot_ip="$(arg robot_ip)"
-    use_fake_hardware="$(arg use_fake_hardware)" />
+    use_fake_hardware="$(arg use_fake_hardware)"
+    fake_sensor_commands="$(arg fake_sensor_commands)"
+    gazebo_effort="$(arg gazebo_effort)"
+    no_prefix="$(arg no_prefix)"
+    arm_prefix=""
+    connected_to="base">
+  </xacro:franka_robot>
 </robot>

File: lbx_robotics/src/lbx_franka_description/urdf/fr3_ros2_control.xacro (robot description, xacro)
@@ -13,9 +13,6 @@
           <param name="robot_ip">${robot_ip}</param>
           <param name="arm_id">${arm_id}</param>
-          <param name="prefix">${arm_id}_</param>
+          <param name="prefix">${arm_id}</param>
           <param name="version">0.1.0</param>
-          <param name="joint_names">${arm_id}_joint1 ${arm_id}_joint2 ${arm_id}_joint3 ${arm_id}_joint4 ${arm_id}_joint5 ${arm_id}_joint6 ${arm_id}_joint7</param>
-          <param name="command_interfaces">position velocity</param>
-          <param name="state_interfaces">position velocity effort</param>
         </xacro:unless>
       </hardware>
